File: conduWIT/conduWIT.kicad_pcb (KiCad board)
At the start: 2 copper layers, 68.6 x 53.3 mm, 8 parts, among them P1 Power, P2 Analog, P3 Digital, P4 Digital, P5 CONN_01X01, P6 CONN_01X01, P7 CONN_01X01, P8 CONN_01X01

Commit message: Updated pin headers
Parts:
- P1, P4: footprint Socket_Arduino_Uno:Socket_Strip_Arduino_1x08 -> conduWIT_parts:Socket_Strip_Arduino_1x08
- P2: footprint Socket_Arduino_Uno:Socket_Strip_Arduino_1x06 -> conduWIT_parts:Socket_Strip_Arduino_1x06
- P3: footprint Socket_Arduino_Uno:Socket_Strip_Arduino_1x10 -> conduWIT_parts:Socket_Strip_Arduino_1x10
